Commit message: Adjust joint origin positions for fins

File: models/tethys.urdf (robot description, URDF)
Before this commit: robot tethys, 4 links, 3 joints
Joints:
- joint horizontal_fins_joint: origin xyz=-0.75 0 0 rpy=0 0 0 -> xyz=-1.05 0 0 rpy=0 0 0
- joint vertical_fins_joint: origin xyz=-0.75 0 0 rpy=0 0 0 -> xyz=-1.05 0 0 rpy=0 0 0
